File: 01_DESIGN/INDEX.kicad_sch (KiCad schematic)
At the start: 0 parts

Commit message: Update project
Other:
- note added: "........."
- note added: "............................................"
- note added: "1"
- note added: "10"
- note added: "11"
- note added: "12"
- note added: "13"
- note added: "14"
- note added: "15"
- note added: "16"
- note added: "17"
- note added: "18"
- note added: "19"
- note added: "2"
- note added: "20"
- note added: "21"
- note added: "22"
- note added: "23"
- note added: "24"
- note added: "25"
- note added: "26"
- note added: "27"
- note added: "28"
- note added: "29"
- note added: "3"
- note added: "30"
- note added: "4"
- note added: "5"
- note added: "6"
- note added: "7"
- note added: "8"
- note added: "9"
- note added: "AVR"
- note added: "BLOCK DIAGRAM"
- note added: "COVER PAGE"
- note added: "INDEX"
- note added: "ISO UART"
- note added: "MCU"
- note added: "POWER"
- note added: "Page"
- note added: "Title"
- note added: "eMMC"
