File: 01_DESIGN/MCU.kicad_sch (KiCad schematic)
At the start: 41 parts, among them J3 USB_B_Micro, J4 Conn_01x08, SW1 SW_DPST_x2, U3 STM32H745ZITx, Y1 Crystal_GND24

Commit message: Update project
Parts:
- removed C31: 100nF, Capacitor_SMD:C_0603_1608Metric, symbol Device:C
Other:
- note removed: "FOR VBAT"
- title: (none) -> MCU

Commit message: Update KiCad project files
Parts:
- BT1: footprint Battery:BatteryHolder_Keystone_3002_1x2032 -> Battery:BatteryHolder_Keystone_1060_1x2032; symbol Device:Battery_Cell -> LABLIB:Battery_Cell
- C10, C11, C12, C13, C14, C15, C16, C18, C19, C20, C22, C23, C24, C25, C26, C27, C28, C29, C30, C32, C33, C34, C5, C6, C7, C8, C9: symbol Device:C -> LABLIB:C
- C17, C21: symbol Device:C_Polarized_US -> LABLIB:C_Polarized_US
- J3: symbol Connector:USB_B_Micro -> LABLIB:USB_B_Micro
- J4: symbol Connector_Generic:Conn_01x08 -> LABLIB:Conn_01x08
- R17, R18, R3, R4, R5: symbol Device:R -> LABLIB:R
- SW1: symbol Switch:SW_DPST_x2 -> LABLIB:SW_DPST_x2
- U3: symbol MCU_ST_STM32H7:STM32H745ZITx -> LABLIB:STM32H745ZITx
- Y1: symbol Device:Crystal_GND24 -> LABLIB:Crystal_GND24
Connections:
- net VDD33USB is gone; now on net +3.3V: C25.1, U3.91 (VDD33_USB)
- net VDD50USB is gone; now on net +3.3V: C26.1, U3.90 (VDD50_USB)
