File: 01_DESIGN/POWER.kicad_sch (KiCad schematic)
At the start: 14 parts, among them J1 Screw_Terminal_01x02, U1 LM2596S-5, U8 TPS7A4533DCQR

Commit message: Update project
Parts:
- added H1, H3: M3, MountingHole:MountingHole_2.7mm_Pad, symbol hex_M3:root_0_mirrored_HEX-M3_hex_M3.IntLib
- added H2, H4: M3, MountingHole:MountingHole_2.7mm_Pad, symbol hex_M3:root_0_HEX-M3_hex_M3.IntLib
- D2: value SS24 -> SS34
- L1: value 44uH -> 47uH
Connections:
- new net SHIELDING: H1.1, H2.1, H3.1, H4.1
Other:
- moved on the sheet: C1, C2, C3, C4, D1, D2, D3, D4, J1, L1, R1, R2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

Commit message: Update KiCad project files
Parts:
- removed U8: TPS7A4533DCQR, Package_TO_SOT_SMD:SOT-223-6, symbol AUSB:CMP-0395-00360-2
- added C31, C60: 100nF, Capacitor_SMD:C_0603_1608Metric, symbol LABLIB:C
- added U2: TPS7A4533DCQR, Package_TO_SOT_SMD:SOT-223-6, symbol LABLIB:TPS7A4533DCQR
- C1, C2, C3, C4: symbol Device:C_Polarized_Small_US -> LABLIB:C_Polarized_Small_US
- D1: symbol Diode:SS34 -> LABLIB:SS34
- D2: symbol Diode:SS24 -> LABLIB:SS24
- H1, H3: symbol hex_M3:root_0_mirrored_HEX-M3_hex_M3.IntLib -> LABLIB:root_0_mirrored_HEX-M3_hex_M3.IntLib
- H2, H4: symbol hex_M3:root_0_HEX-M3_hex_M3.IntLib -> LABLIB:root_0_HEX-M3_hex_M3.IntLib
- J1: symbol Connector:Screw_Terminal_01x02 -> LABLIB:Screw_Terminal_01x02
- L1: symbol Device:L -> LABLIB:L
- POWER_LED_12V-5V1: renamed from D3; symbol Device:LED -> LABLIB:LED
- POWER_LED_5V-3.3V1: renamed from D4; symbol Device:LED -> LABLIB:LED
- R1, R2: symbol Device:R -> LABLIB:R
- U1: symbol Regulator_Switching:LM2596S-5 -> LABLIB:LM2596S-5
Connections:
- net SHIELDING is gone; now on net GND: H1.1, H2.1, H3.1, H4.1
- net +12V: now also J1.1 (Pin_1), C31.1; no longer J1.2 (Pin_2)
- net +3.3V: now also U2.4 (OUT), U2.5 (SENSE)
- net +5V: now also C60.1, U2.1 (~{SHDN}), U2.2 (IN)
- net GND: now also J1.2 (Pin_2), C31.2, C60.2, U2.3 (GND), U2.6 (GND); no longer J1.1 (Pin_1)
Other:
- moved on the sheet: C1, J1, POWER_LED_12V-5V1, R1
